Commit message: 🐛 将urdf模型和xml模型与legged_control一致

File: resources/robots/go1/urdf/go1.urdf (robot description, URDF)
Before this commit: robot go1_description, 23 links, 22 joints
Links:
- link FL_calf: mass 0.158015 -> 0.135862
- link FL_hip: mass 0.510299 -> 0.591
- link FL_thigh: mass 0.898919 -> 0.92
- link FR_calf: mass 0.158015 -> 0.135862
- link FR_hip: mass 0.510299 -> 0.591
- link FR_thigh: mass 0.898919 -> 0.92
- link RL_calf: mass 0.158015 -> 0.135862
- link RL_hip: mass 0.510299 -> 0.591
- link RL_thigh: mass 0.898919 -> 0.92
- link RR_calf: mass 0.158015 -> 0.135862
- link RR_hip: mass 0.510299 -> 0.591
- link RR_thigh: mass 0.898919 -> 0.92
- link imu_link: mass 0.001 -> 0.01
- link trunk: mass 4.8 -> 5.29
Joints:
- joint FL_calf_joint: limit lower=-2.69653369433 upper=-0.916297857297 effort=33.5 velocity=28 -> lower=-2.818 upper=-0.888 effort=35.55 velocity=20.06
- joint FL_hip_joint: limit lower=-0.802851455917 upper=0.802851455917 effort=23.7 velocity=50 -> lower=-0.863 upper=0.863 effort=23.7 velocity=30.1
- joint FL_thigh_joint: limit lower=-1.0471975512 upper=4.18879020479 effort=23.7 velocity=28 -> lower=-0.686 upper=4.501 effort=23.7 velocity=30.1
- joint FR_calf_joint: limit lower=-2.69653369433 upper=-0.916297857297 effort=33.5 velocity=28 -> lower=-2.818 upper=-0.888 effort=35.55 velocity=20.06
- joint FR_hip_joint: limit lower=-0.802851455917 upper=0.802851455917 effort=23.7 velocity=50 -> lower=-0.863 upper=0.863 effort=23.7 velocity=30.1
- joint FR_thigh_joint: limit lower=-1.0471975512 upper=4.18879020479 effort=23.7 velocity=28 -> lower=-0.686 upper=4.501 effort=23.7 velocity=30.1
- joint RL_calf_joint: limit lower=-2.69653369433 upper=-0.916297857297 effort=33.5 velocity=28 -> lower=-2.818 upper=-0.888 effort=35.55 velocity=20.06
- joint RL_hip_joint: limit lower=-0.802851455917 upper=0.802851455917 effort=23.7 velocity=50 -> lower=-0.863 upper=0.863 effort=23.7 velocity=30.1
- joint RL_thigh_joint: limit lower=-1.0471975512 upper=4.18879020479 effort=23.7 velocity=28 -> lower=-0.686 upper=4.501 effort=23.7 velocity=30.1
- joint RR_calf_joint: limit lower=-2.69653369433 upper=-0.916297857297 effort=33.5 velocity=28 -> lower=-2.818 upper=-0.888 effort=35.55 velocity=20.06
- joint RR_hip_joint: limit lower=-0.802851455917 upper=0.802851455917 effort=23.7 velocity=50 -> lower=-0.863 upper=0.863 effort=23.7 velocity=30.1
- joint RR_thigh_joint: limit lower=-1.0471975512 upper=4.18879020479 effort=23.7 velocity=28 -> lower=-0.686 upper=4.501 effort=23.7 velocity=30.1
- joint imu_joint: origin xyz=-0.01592 -0.06659 -0.00617 rpy=0 0 0 -> xyz=0 0 0 rpy=0 0 0

Commit message: 🎨 用dream的模型和初始关节角，feet_air_time=0.02

File: resources/robots/go1/urdf/go1.urdf (robot description, URDF)
Before this commit: robot go1_description, 23 links, 22 joints
Links:
- link FL_calf: mass 0.135862 -> 0.158015
- link FL_hip: mass 0.591 -> 0.510299
- link FL_thigh: mass 0.92 -> 0.898919
- link FR_calf: mass 0.135862 -> 0.158015
- link FR_hip: mass 0.591 -> 0.510299
- link FR_thigh: mass 0.92 -> 0.898919
- link RL_calf: mass 0.135862 -> 0.158015
- link RL_hip: mass 0.591 -> 0.510299
- link RL_thigh: mass 0.92 -> 0.898919
- link RR_calf: mass 0.135862 -> 0.158015
- link RR_hip: mass 0.591 -> 0.510299
- link RR_thigh: mass 0.92 -> 0.898919
- link imu_link: mass 0.01 -> 0.001
- link trunk: mass 5.29 -> 4.8
Joints:
- joint FL_calf_joint: limit lower=-2.818 upper=-0.888 effort=35.55 velocity=20.06 -> lower=-2.69653369433 upper=-0.916297857297 effort=33.5 velocity=28
- joint FL_hip_joint: limit lower=-0.863 upper=0.863 effort=23.7 velocity=30.1 -> lower=-0.802851455917 upper=0.802851455917 effort=33.5 velocity=50
- joint FL_thigh_joint: limit lower=-0.686 upper=4.501 effort=23.7 velocity=30.1 -> lower=-1.0471975512 upper=4.18879020479 effort=33.5 velocity=28
- joint FR_calf_joint: limit lower=-2.818 upper=-0.888 effort=35.55 velocity=20.06 -> lower=-2.69653369433 upper=-0.916297857297 effort=33.5 velocity=28
- joint FR_hip_joint: limit lower=-0.863 upper=0.863 effort=23.7 velocity=30.1 -> lower=-0.802851455917 upper=0.802851455917 effort=33.5 velocity=50
- joint FR_thigh_joint: limit lower=-0.686 upper=4.501 effort=23.7 velocity=30.1 -> lower=-1.0471975512 upper=4.18879020479 effort=33.5 velocity=28
- joint RL_calf_joint: limit lower=-2.818 upper=-0.888 effort=35.55 velocity=20.06 -> lower=-2.69653369433 upper=-0.916297857297 effort=33.5 velocity=28
- joint RL_hip_joint: limit lower=-0.863 upper=0.863 effort=23.7 velocity=30.1 -> lower=-0.802851455917 upper=0.802851455917 effort=33.5 velocity=50
- joint RL_thigh_joint: limit lower=-0.686 upper=4.501 effort=23.7 velocity=30.1 -> lower=-1.0471975512 upper=4.18879020479 effort=33.5 velocity=28
- joint RR_calf_joint: limit lower=-2.818 upper=-0.888 effort=35.55 velocity=20.06 -> lower=-2.69653369433 upper=-0.916297857297 effort=33.5 velocity=28
- joint RR_hip_joint: limit lower=-0.863 upper=0.863 effort=23.7 velocity=30.1 -> lower=-0.802851455917 upper=0.802851455917 effort=33.5 velocity=50
- joint RR_thigh_joint: limit lower=-0.686 upper=4.501 effort=23.7 velocity=30.1 -> lower=-1.0471975512 upper=4.18879020479 effort=33.5 velocity=28
- joint imu_joint: origin xyz=0 0 0 rpy=0 0 0 -> xyz=-0.01592 -0.06659 -0.00617 rpy=0 0 0
